Commit message: Lidar model changes

File: bme_ros_micromouse/urdf/umouse_robot.xacro (robot description, xacro)
@@ -64,5 +64,5 @@
   <!-- STEP 2 - Wheels -->
   <joint type="continuous" name="left_wheel_joint">
-    <origin xyz="0 0.15 0" rpy="0 0 0"/>
+    <origin xyz="0 0.02 0" rpy="0 0 0"/>
     <child link="left_wheel"/>
     <parent link="base_link"/>
@@ -97,5 +97,5 @@
   </link>
   <joint type="continuous" name="right_wheel_joint">
-    <origin xyz="0 -0.15 0" rpy="0 0 0"/>
+    <origin xyz="0 -0.02 0" rpy="0 0 0"/>
     <child link="right_wheel"/>
     <parent link="base_link"/>
@@ -141,5 +141,5 @@
 <!-- Lidar -->
   <joint type="fixed" name="scan_joint">
-    <origin xyz="0.0 0 0.15" rpy="0 0 0"/>
+    <origin xyz="0.0 0 0.02" rpy="0 0 0"/>
     <child link="scan_link"/>
     <parent link="base_link"/>

Commit message: Modify robot xacro file

File: bme_ros_micromouse/urdf/umouse_robot.xacro (robot description, xacro)
@@ -38,25 +38,25 @@
     </visual>
     <collision name='rear_caster_collision'>
-      <origin xyz="-0.15 0 -0.05" rpy=" 0 0 0"/>
+      <origin xyz="-0.03 0 -0.005" rpy=" 0 0 0"/>
       <geometry>
-        <sphere radius="0.0499"/>
+        <sphere radius="0.0079"/>
       </geometry>
     </collision>
     <visual name='rear_caster_visual'>
-      <origin xyz="-0.15 0 -0.05" rpy=" 0 0 0"/>
+      <origin xyz="-0.03 0 -0.005" rpy=" 0 0 0"/>
       <geometry>
-        <sphere radius="0.05"/>
+        <sphere radius="0.008"/>
       </geometry>
     </visual>
     <collision name='front_caster_collision'>
-      <origin xyz="0.15 0 -0.05" rpy=" 0 0 0"/>
+      <origin xyz="0.04 0 -0.005" rpy=" 0 0 0"/>
       <geometry>
-        <sphere radius="0.0499"/>
+        <sphere radius="0.0079"/>
       </geometry>
     </collision>
     <visual name='front_caster_visual'>
-      <origin xyz="0.15 0 -0.05" rpy=" 0 0 0"/>
+      <origin xyz="0.04 0 -0.005" rpy=" 0 0 0"/>
       <geometry>
-        <sphere radius="0.05"/>
+        <sphere radius="0.008"/>
       </geometry>
     </visual>

Commit message: Bug fix in robot xacro file

File: bme_ros_micromouse/urdf/umouse_robot.xacro (robot description, xacro)
@@ -26,5 +26,6 @@
       <origin xyz="0 0 0" rpy=" 0 0 0"/>
       <geometry>
-        <box size=".4 .2 .1"/>
+        <box size=".1 .03 .016"/>
+        <!--box size=".1 .06 .016"/-->
       </geometry>
     </collision>
@@ -38,5 +39,5 @@
     </visual>
     <collision name='rear_caster_collision'>
-      <origin xyz="-0.03 0 -0.005" rpy=" 0 0 0"/>
+      <origin xyz="-0.04 0 -0.005" rpy=" 0 0 0"/>
       <geometry>
         <sphere radius="0.0079"/>
@@ -44,5 +45,5 @@
     </collision>
     <visual name='rear_caster_visual'>
-      <origin xyz="-0.03 0 -0.005" rpy=" 0 0 0"/>
+      <origin xyz="-0.04 0 -0.005" rpy=" 0 0 0"/>
       <geometry>
         <sphere radius="0.008"/>
@@ -50,5 +51,5 @@
     </visual>
     <collision name='front_caster_collision'>
-      <origin xyz="0.04 0 -0.005" rpy=" 0 0 0"/>
+      <origin xyz="0.025 0 -0.005" rpy=" 0 0 0"/>
       <geometry>
         <sphere radius="0.0079"/>
@@ -56,5 +57,5 @@
     </collision>
     <visual name='front_caster_visual'>
-      <origin xyz="0.04 0 -0.005" rpy=" 0 0 0"/>
+      <origin xyz="0.025 0 -0.005" rpy=" 0 0 0"/>
       <geometry>
         <sphere radius="0.008"/>
@@ -82,7 +83,7 @@
     </inertial>
     <collision name='collision'>
-      <origin xyz="0 0 0" rpy="0 1.5707 1.5707"/>
+      <origin xyz="0 0 0" rpy="0 1.5707 1.57070"/>
       <geometry>
-        <cylinder radius=".1" length=".05"/>
+        <cylinder radius=".015" length=".003"/>
       </geometry>
     </collision>
@@ -117,5 +118,5 @@
       <origin xyz="0 0 0" rpy="0 1.5707 1.5707"/>
       <geometry>
-        <cylinder radius=".1" length=".05"/>
+        <cylinder radius=".015" length=".003"/>
       </geometry>
     </collision>
@@ -159,5 +160,5 @@
       <origin xyz="0 0 0" rpy="0 0 0"/>
       <geometry>
-        <box size=".1 .1 .1"/>
+        <box size=".03 .03 .03"/>
       </geometry>
     </collision>

Commit message: Bugfix

File: bme_ros_micromouse/urdf/umouse_robot.xacro (robot description, xacro)
@@ -36,10 +36,10 @@
         <mesh filename = "package://bme_ros_micromouse/meshes/body.dae"/>
       </geometry>
-      <material name="pink"/>
+      <material name="orange"/>
     </visual>
     <collision name='rear_caster_collision'>
       <origin xyz="-0.04 0 -0.005" rpy=" 0 0 0"/>
       <geometry>
-        <sphere radius="0.0079"/>
+        <sphere radius="0.0099"/>
       </geometry>
     </collision>
@@ -47,5 +47,5 @@
       <origin xyz="-0.04 0 -0.005" rpy=" 0 0 0"/>
       <geometry>
-        <sphere radius="0.008"/>
+        <sphere radius="0.01"/>
       </geometry>
     </visual>
@@ -53,5 +53,5 @@
       <origin xyz="0.025 0 -0.005" rpy=" 0 0 0"/>
       <geometry>
-        <sphere radius="0.0079"/>
+        <sphere radius="0.0099"/>
       </geometry>
     </collision>
@@ -59,5 +59,5 @@
       <origin xyz="0.025 0 -0.005" rpy=" 0 0 0"/>
       <geometry>
-        <sphere radius="0.008"/>
+        <sphere radius="0.01"/>
       </geometry>
     </visual>
@@ -141,5 +141,5 @@
   </gazebo-->
 <!-- Lidar -->
-  <joint type="fixed" name="scan_joint">
+  <!--joint type="fixed" name="scan_joint">
     <origin xyz="0.0 0 0.02" rpy="0 0 0"/>
     <child link="scan_link"/>
@@ -169,4 +169,4 @@
       </geometry>
     </visual>
-  </link>
+  </link-->
 </robot>

Commit message: Change robot model

File: bme_ros_micromouse/urdf/umouse_robot.xacro (robot description, xacro)
@@ -15,10 +15,10 @@
     <pose>0 0 0.1 0 0 0</pose>
     <inertial>
-      <mass value="15.0"/>
+      <mass value="3.75"/>
       <origin xyz="0.0 0 0" rpy=" 0 0 0"/>
       <inertia
-          ixx="0.1" ixy="0" ixz="0"
-          iyy="0.1" iyz="0"
-          izz="0.1"
+          ixx="0.01" ixy="0" ixz="0"
+          iyy="0.01" iyz="0"
+          izz="0.01"
       />
     </inertial>
@@ -26,6 +26,5 @@
       <origin xyz="0 0 0" rpy=" 0 0 0"/>
       <geometry>
-        <box size=".1 .03 .016"/>
-        <!--box size=".1 .06 .016"/-->
+        <box size=".1 .05 .025"/>
       </geometry>
     </collision>
@@ -33,5 +32,4 @@
       <origin xyz="0 0 0" rpy=" 0 0 0"/>
       <geometry>
-        <!--box size=".4 .2 .1"/-->
         <mesh filename = "package://bme_ros_micromouse/meshes/body.dae"/>
       </geometry>
@@ -39,25 +37,25 @@
     </visual>
     <collision name='rear_caster_collision'>
-      <origin xyz="-0.04 0 -0.005" rpy=" 0 0 0"/>
+      <origin xyz="-0.0375 0 -0.0125" rpy=" 0 0 0"/>
       <geometry>
-        <sphere radius="0.0099"/>
+        <sphere radius="0.0124"/>
       </geometry>
     </collision>
     <visual name='rear_caster_visual'>
-      <origin xyz="-0.04 0 -0.005" rpy=" 0 0 0"/>
+      <origin xyz="-0.0375 0 -0.0125" rpy=" 0 0 0"/>
       <geometry>
-        <sphere radius="0.01"/>
+        <sphere radius="0.0125"/>
       </geometry>
     </visual>
     <collision name='front_caster_collision'>
-      <origin xyz="0.025 0 -0.005" rpy=" 0 0 0"/>
+      <origin xyz="0.0375 0 -0.0125" rpy=" 0 0 0"/>
       <geometry>
-        <sphere radius="0.0099"/>
+        <sphere radius="0.0124"/>
       </geometry>
     </collision>
     <visual name='front_caster_visual'>
-      <origin xyz="0.025 0 -0.005" rpy=" 0 0 0"/>
+      <origin xyz="0.0375 0 -0.0125" rpy=" 0 0 0"/>
       <geometry>
-        <sphere radius="0.01"/>
+        <sphere radius="0.0125"/>
       </geometry>
     </visual>
@@ -65,5 +63,5 @@
   <!-- STEP 2 - Wheels -->
   <joint type="continuous" name="left_wheel_joint">
-    <origin xyz="0 0.02 0" rpy="0 0 0"/>
+    <origin xyz="0 0.0375 0" rpy="0 0 0"/>
     <child link="left_wheel"/>
     <parent link="base_link"/>
@@ -74,10 +72,10 @@
   <link name='left_wheel'>
     <inertial>
-      <mass value="5.0"/>
+      <mass value="1.25"/>
       <origin xyz="0 0 0" rpy="0 1.5707 1.5707"/>
       <inertia
-          ixx="0.1" ixy="0" ixz="0"
-          iyy="0.1" iyz="0"
-          izz="0.1"
+          ixx="0.01" ixy="0" ixz="0"
+          iyy="0.01" iyz="0"
+          izz="0.01"
       />
     </inertial>
@@ -85,5 +83,5 @@
       <origin xyz="0 0 0" rpy="0 1.5707 1.57070"/>
       <geometry>
-        <cylinder radius=".015" length=".003"/>
+        <cylinder radius=".025" length=".0125"/>
       </geometry>
     </collision>
@@ -91,5 +89,4 @@
       <origin xyz="0 0 0" rpy="0 1.5707 1.5707"/>
       <geometry>
-        <!--cylinder radius=".1" length=".05"/-->
         <mesh filename = "package://bme_ros_micromouse/meshes/wheel.dae"/>
       </geometry>
@@ -98,5 +95,5 @@
   </link>
   <joint type="continuous" name="right_wheel_joint">
-    <origin xyz="0 -0.02 0" rpy="0 0 0"/>
+    <origin xyz="0 -0.0375 0" rpy="0 0 0"/>
     <child link="right_wheel"/>
     <parent link="base_link"/>
@@ -107,10 +104,10 @@
   <link name='right_wheel'>
     <inertial>
-      <mass value="5.0"/>
+      <mass value="1.25"/>
       <origin xyz="0 0 0" rpy="0 1.5707 1.5707"/>
       <inertia
-          ixx="0.1" ixy="0" ixz="0"
-          iyy="0.1" iyz="0"
-          izz="0.1"
+          ixx="0.01" ixy="0" ixz="0"
+          iyy="0.01" iyz="0"
+          izz="0.01"
       />
     </inertial>
@@ -118,5 +115,5 @@
       <origin xyz="0 0 0" rpy="0 1.5707 1.5707"/>
       <geometry>
-        <cylinder radius=".015" length=".003"/>
+        <cylinder radius=".025" length=".0125"/>
       </geometry>
     </collision>
@@ -124,5 +121,4 @@
       <origin xyz="0 0 0" rpy="0 1.5707 1.5707"/>
       <geometry>
-        <!--cylinder radius=".1" length=".05"/-->
         <mesh filename = "package://bme_ros_micromouse/meshes/wheel.dae"/>
       </geometry>
@@ -141,6 +137,6 @@
   </gazebo-->
 <!-- Lidar -->
-  <!--joint type="fixed" name="scan_joint">
-    <origin xyz="0.0 0 0.02" rpy="0 0 0"/>
+  <joint type="fixed" name="scan_joint">
+    <origin xyz="0.0 0 0.031" rpy="0 0 0"/>
     <child link="scan_link"/>
     <parent link="base_link"/>
@@ -160,5 +156,5 @@
       <origin xyz="0 0 0" rpy="0 0 0"/>
       <geometry>
-        <box size=".03 .03 .03"/>
+        <box size=".025 .025 .025"/>
       </geometry>
     </collision>
@@ -169,4 +165,4 @@
       </geometry>
     </visual>
-  </link-->
+  </link>
 </robot>

Commit message: Need fix

File: bme_ros_micromouse/urdf/umouse_robot.xacro (robot description, xacro)
@@ -126,14 +126,12 @@
     </visual>
   </link>
-  <!-- STEP 4 - Gazebo colors -->
-  <!--gazebo reference="left_wheel">
-    <material>Gazebo/Green</material>
-  </gazebo>
-  <gazebo reference="right_wheel">
-    <material>Gazebo/Green</material>
-  </gazebo>
-  <gazebo reference="base_link">
-    <material>Gazebo/Pink</material>
-  </gazebo-->
+  <!-- IMU -->
+  <joint name="imu_joint" type="fixed">
+    <origin xyz="0 0 0" rpy="0 0 0" />
+    <parent link="base_link"/>
+    <child link="imu_link" />
+  </joint>
+  <link name="imu_link">
+  </link>
 <!-- Lidar -->
   <joint type="fixed" name="scan_joint">
